File: bowden-toolhead.kicad_pcb (KiCad board)
At the start: 2 copper layers, 34 x 50 mm, 87 parts, among them J101 918-418K2022Y40004, J102 POWER, J103 PARTFAN_A, J104 PARTFAN_B, J105 CANBUS, J106 HEFAN, J107 HEATER, J108 THERM0, J201 STM32-SWD-POGO, Q101 AO3400A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

Commit message: work on layout
Parts:
- moved J108 93.1 mm to (137.7, 127.6), turned to 180 degrees
- moved Q101 87.9 mm to (61.3, 52.2), turned to 90 degrees
- moved U101 81.9 mm to (140.6, 30.4)
- moved R203 58.7 mm to (112.5, 94.8), turned to 90 degrees
- moved C122 51.9 mm to (139.7, 113.9)
- moved R122 51.2 mm to (141.7, 113.9)
- moved R204 47.6 mm to (110.9, 94.8), turned to 90 degrees
- moved Q104 23.2 mm to (97.5, 67.7)
- moved R119 21.6 mm to (139.7, 118.5)
- moved U202 13.4 mm to (97.1, 91.4), turned to -90 degrees
- moved J201 7.88 mm to (117.7, 98.2), turned to 90 degrees
- moved R120 7.46 mm to (141.7, 118.5), turned to 180 degrees
- moved D105 6.48 mm to (140.7, 116.2)
- moved R205 5.88 mm to (165.0, 93.2)
- moved U201 4.88 mm to (102.8, 102.5), turned to -90 degrees
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Routing:
- net THERM0: track 0.00 -> 0.96 mm

Commit message: Auto-commit Mon Feb 13 12:20:09 EST 2023
Parts:
- moved R116 84.0 mm to (97.9, 103.9), turned to -90 degrees
- moved D107 55.8 mm to (136.8, 116.2), turned to 180 degrees
- moved R111 41.9 mm to (95.0, 73.9), turned to 180 degrees
- moved R118 28.6 mm to (95.9, 107.4), turned to 180 degrees
- moved SW101 0.39 mm to (97.2, 104.5)
Changed lines of the file:
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@@
   )
   (footprint "Package_TO_SOT_SMD:SOT-23" (layer "F.Cu")
-    (at 83.5406 99.3902)
+    (at 136.7536 116.2304 180)
     (descr "SOT, 3 Pin (https://www.jedec.org/system/files/docs/to-236h.pdf variant AB), generated with kicad-footprint-generator ipc_gullwing_generator.py")
     (tags "SOT TO_SOT_SMD")
@@
     (property "Sheetname" "")
     (attr smd)
-    (fp_text reference "D107" (at 0 -2.4) (layer "F.SilkS")
+    (fp_text reference "D107" (at 2.667 0.1016 90) (layer "F.SilkS")
       (effects (font (size 1 1) (thickness 0.15)))
     )
@@
     (fp_line (start 0.65 -1.45) (end 0.65 1.45) (layer "F.Fab") (width 0.1))
     (fp_line (start 0.65 1.45) (end -0.65 1.45) (layer "F.Fab") (width 0.1))
-    (pad "1" smd roundrect (at -0.9375 -0.95) (size 1.475 0.6) (layers "F.Cu" "F.Paste" "F.Mask") (roundrect_rratio 0.25)
+    (pad "1" smd roundrect (at -0.9375 -0.95 180) (size 1.475 0.6) (layers "F.Cu" "F.Paste" "F.Mask") (roundrect_rratio 0.25)
       (net 10 "THERM0_MCU") (pinfunction "A1") (pintype "passive"))
-    (pad "2" smd roundrect (at -0.9375 0.95) (size 1.475 0.6) (layers "F.Cu" "F.Paste" "F.Mask") (roundrect_rratio 0.25)
+    (pad "2" smd roundrect (at -0.9375 0.95 180) (size 1.475 0.6) (layers "F.Cu" "F.Paste" "F.Mask") (roundrect_rratio 0.25)
       (net 2 "GND") (pinfunction "A2") (pintype "passive"))
-    (pad "3" smd roundrect (at 0.9375 0) (size 1.475 0.6) (layers "F.Cu" "F.Paste" "F.Mask") (roundrect_rratio 0.25))
+    (pad "3" smd roundrect (at 0.9375 0 180) (size 1.475 0.6) (layers "F.Cu" "F.Paste" "F.Mask") (roundrect_rratio 0.25))
     (model "${KICAD6_3DMODEL_DIR}/Package_TO_SOT_SMD.3dshapes/SOT-23.wrl"
       (offset (xyz 0 0 0))
@@
   )
   (footprint "Resistor_SMD:R_0402_1005Metric" (layer "F.Cu")
-    (at 173.9424 68.2634)
+    (at 97.917 103.9114 -90)
     (descr "Resistor SMD 0402 (1005 Metric), square (rectangular) end terminal, IPC_7351 nominal, (Body size source: IPC-SM-782 page 72, https://www.pcb-3d.com/wordpress/wp-content/uploads/ipc-sm-782a_amendment_1_and_2.pdf), generated with kicad-footprint-generator")
     (tags "resistor")
@@
     (property "Sheetname" "")
     (attr smd)
-    (fp_text reference "R116" (at 0 -1.17) (layer "F.SilkS")
+    (fp_text reference "R116" (at -2.794 -0.0508 90) (layer "F.SilkS")
       (effects (font (size 1 1) (thickness 0.15)))
     )
-    (fp_text value "DNP" (at 0 1.17) (layer "F.Fab")
+    (fp_text value "DNP" (at 0 1.17 90) (layer "F.Fab")
       (effects (font (size 1 1) (thickness 0.15)))
     )
-    (fp_text user "${REFERENCE}" (at 0 0) (layer "F.Fab")
+    (fp_text user "${REFERENCE}" (at 0 0 90) (layer "F.Fab")
       (effects (font (size 0.26 0.26) (thickness 0.04)))
     )
@@
     (fp_line (start -0.525 0.27) (end -0.525 -0.27) (layer "F.Fab") (width 0.1))
     (fp_line (start 0.525 -0.27) (end 0.525 0.27) (layer "F.Fab") (width 0.1))
-    (pad "1" smd roundrect (at -0.51 0) (size 0.54 0.64) (layers "F.Cu" "F.Paste" "F.Mask") (roundrect_rratio 0.25)
+    (pad "1" smd roundrect (at -0.51 0 270) (size 0.54 0.64) (layers "F.Cu" "F.Paste" "F.Mask") (roundrect_rratio 0.25)
       (net 8 "+3V3") (pintype "passive"))
-    (pad "2" smd roundrect (at 0.51 0) (size 0.54 0.64) (layers "F.Cu" "F.Paste" "F.Mask") (roundrect_rratio 0.25)
+    (pad "2" smd roundrect (at 0.51 0 270) (size 0.54 0.64) (layers "F.Cu" "F.Paste" "F.Mask") (roundrect_rratio 0.25)
       (net 9 "XEND") (pintype "passive"))
     (model "${KICAD6_3DMODEL_DIR}/Resistor_SMD.3dshapes/R_0402_1005Metric.wrl"
@@
   )
   (footprint "Resistor_SMD:R_0402_1005Metric" (layer "F.Cu")
-    (at 120.4124 122.0934)
+    (at 95.8596 107.4166 180)
     (descr "Resistor SMD 0402 (1005 Metric), square (rectangular) end terminal, IPC_7351 nominal, (Body size source: IPC-SM-782 page 72, https://www.pcb-3d.com/wordpress/wp-content/uploads/ipc-sm-782a_amendment_1_and_2.pdf), generated with kicad-footprint-generator")
     (tags "resistor")
@@
     (property "Sheetname" "")
     (attr smd)
-    (fp_text reference "R118" (at 0 -1.17) (layer "F.SilkS")
+    (fp_text reference "R118" (at -2.9464 -0.0254) (layer "F.SilkS")
       (effects (font (size 1 1) (thickness 0.15)))
     )
@@
     (fp_line (start -0.525 0.27) (end -0.525 -0.27) (layer "F.Fab") (width 0.1))
     (fp_line (start 0.525 -0.27) (end 0.525 0.27) (layer "F.Fab") (width 0.1))
-    (pad "1" smd roundrect (at -0.51 0) (size 0.54 0.64) (layers "F.Cu" "F.Paste" "F.Mask") (roundrect_rratio 0.25)
+    (pad "1" smd roundrect (at -0.51 0 180) (size 0.54 0.64) (layers "F.Cu" "F.Paste" "F.Mask") (roundrect_rratio 0.25)
       (net 9 "XEND") (pintype "passive"))
-    (pad "2" smd roundrect (at 0.51 0) (size 0.54 0.64) (layers "F.Cu" "F.Paste" "F.Mask") (roundrect_rratio 0.25)
+    (pad "2" smd roundrect (at 0.51 0 180) (size 0.54 0.64) (layers "F.Cu" "F.Paste" "F.Mask") (roundrect_rratio 0.25)
       (net 49 "Net-(R118-Pad2)") (pintype "passive"))
     (model "${KICAD6_3DMODEL_DIR}/Resistor_SMD.3dshapes/R_0402_1005Metric.wrl"
@@
   )
   (footprint "Resistor_SMD:R_0402_1005Metric" (layer "F.Cu")
-    (at 95.631 115.7986)
+    (at 94.9706 73.8886 180)
     (descr "Resistor SMD 0402 (1005 Metric), square (rectangular) end terminal, IPC_7351 nominal, (Body size source: IPC-SM-782 page 72, https://www.pcb-3d.com/wordpress/wp-content/uploads/ipc-sm-782a_amendment_1_and_2.pdf), generated with kicad-footprint-generator")
     (tags "resistor")
@@
     (property "Sheetname" "")
     (attr smd)
-    (fp_text reference "R111" (at 0 -1.17) (layer "F.SilkS")
+    (fp_text reference "R111" (at -2.8194 -0.0254) (layer "F.SilkS")
       (effects (font (size 1 1) (thickness 0.15)))
     )
@@
     (fp_line (start 0.525 0.27) (end -0.525 0.27) (layer "F.Fab") (width 0.1))
     (fp_line (start -0.525 0.27) (end -0.525 -0.27) (layer "F.Fab") (width 0.1))
-    (pad "1" smd roundrect (at -0.51 0) (size 0.54 0.64) (layers "F.Cu" "F.Paste" "F.Mask") (roundrect_rratio 0.25)
+    (pad "1" smd roundrect (at -0.51 0 180) (size 0.54 0.64) (layers "F.Cu" "F.Paste" "F.Mask") (roundrect_rratio 0.25)
       (net 48 "Net-(R111-Pad1)") (pintype "passive"))
-    (pad "2" smd roundrect (at 0.51 0) (size 0.54 0.64) (layers "F.Cu" "F.Paste" "F.Mask") (roundrect_rratio 0.25)
+    (pad "2" smd roundrect (at 0.51 0 180) (size 0.54 0.64) (layers "F.Cu" "F.Paste" "F.Mask") (roundrect_rratio 0.25)
       (net 41 "Net-(Q104-Pad1)") (pintype "passive"))
     (model "${KICAD6_3DMODEL_DIR}/Resistor_SMD.3dshapes/R_0402_1005Metric.wrl"
@@
   )
   (footprint "matei:D3SH-boss" (layer "F.Cu")
-    (at 96.8502 104.4956 90)
-    (descr "Unnamed StepUp generated footprint")
+    (at 97.2411 104.4956 90)
+    (descr "D3SH StepUp generated footprint")
     (property "Sheetfile" "File: bowden-toolhead.kicad_sch")
     (property "Sheetname" "")
@@
     (fp_circle (center 0 -0.8) (end -0.35 -0.8) (layer "Edge.Cuts") (width 0.15) (fill none))
     (fp_circle (center 0 -2.8) (end -0.35 -2.8) (layer "Edge.Cuts") (width 0.15) (fill none))
-    (fp_line (start -1.5 0) (end -1.5 -3.3) (layer "F.Fab") (width 0.1))
-    (fp_line (start 1.5 0) (end -1.5 0) (layer "F.Fab") (width 0.1))
-    (fp_line (start -1.5 -3.3) (end 1.5 -3.3) (layer "F.Fab") (width 0.1))
-    (fp_line (start 1.5 -3.3) (end 1.5 0) (layer "F.Fab") (width 0.1))
+    (fp_line (start 1.5 0.075) (end -1.5 0.075) (layer "F.CrtYd") (width 0.1))
+    (fp_line (start 1.5 -3.725) (end 1.5 0.075) (layer "F.CrtYd") (width 0.1))
+    (fp_line (start -1.5 -3.725) (end 1.5 -3.725) (layer "F.CrtYd") (width 0.1))
+    (fp_line (start -1.5 0.075) (end -1.5 -3.725) (layer "F.CrtYd") (width 0.1))
     (pad "1" smd rect (at -1.65 -1.65 90) (size 1.1 1.1) (layers "F.Cu" "F.Paste" "F.Mask")
       (net 49 "Net-(R118-Pad2)") (pinfunction "A") (pintype "passive"))
     (pad "2" smd rect (at 1.65 -1.575 90) (size 1.1 0.95) (layers "F.Cu" "F.Paste" "F.Mask")
       (net 2 "GND") (pinfunction "B") (pintype "passive"))
-    (model "/Users/mateijordache/Documents/KiCad/5.99/footprints/matei.pretty/Unnamed.wrl"
+    (model "/Users/mateijordache/Documents/KiCad/6.0/footprints/matei.pretty/D3SH.wrl"
       (offset (xyz 0 0 0))
       (scale (xyz 1 1 1))
@@
       (effects (font (size 1 1) (thickness 0.15)))
     )
-    (fp_text value "PCB" (at -12.7 2.54) (layer "F.SilkS")
+    (fp_text value "PCB" (at -16.0966 1.0712) (layer "F.SilkS")
       (effects (font (size 1 1) (thickness 0.15)))
     )
@@
     )
   )
-  (group "" (id e8e6af59-9a32-432e-85a6-fd36d82173cb)
+  (group "" (id c3ea1e4d-71e4-43e5-8548-9b15d3106732)
     (members
       0da60ca3-3d70-46e3-9615-0dfb471ab81a
+      1d519bf4-5a7c-45f9-90b0-214cf29fb5fd
       2d956407-b7fc-4417-a03c-a7366783ddb8
       36e92712-d287-4f70-b3a2-8aec469d2ec6
